Commit message: Fix styling
Mega commit

File: tm_description/xacro/macro.materials.xacro (robot description, xacro)
@@ -1,44 +1,44 @@
 <?xml version="1.0"?>
 <robot xmlns:xacro="http://www.ros.org/wiki/xacro">
-	<xacro:macro name="tmr_materials">
-		<material name="none">
-			<color rgba="0.0 0.0 0.0 1.0" />
-		</material>
-		<material name="lightgrey">
-			<color rgba="0.5 0.5 0.5 1.0" />
-		</material>
-		<material name="grey">
-			<color rgba="0.75 0.75 0.75 1.0" />
-		</material>
-		<material name="white">
-			<color rgba="0.95 0.95 0.95 1.0" />
-		</material>
-		<material name="red">
-			<color rgba="0.95 0.0 0.0 1.0" />
-		</material>
-		<material name="orange">
-			<color rgba="1.0 0.5 0.0 1.0" />
-		</material>
-		<material name="yellow">
-			<color rgba="1.0 1.0 0.0 1.0" />
-		</material>
-		<material name="green">
-			<color rgba="0.0 1.0 0.0 1.0" />
-		</material>
-		<material name="blue">
-			<color rgba="0.0 0.0 1.0 1.0" />
-		</material>
-		<material name="indigo">
-			<color rgba="0.3 0.3 0.6 1.0" />
-		</material>
-		<material name="violet">
-			<color rgba="0.6 0.0 1.0 1.0" />
-		</material>
-		<material name="black">
-			<color rgba="0.0 0.0 0.0 1.0" />
-		</material>
-		<material name="darkolive">
-			<color rgba="0.3 0.3 0.25 1.0" />
-		</material>
-	</xacro:macro>
+  <xacro:macro name="tmr_materials">
+    <material name="none">
+      <color rgba="0.0 0.0 0.0 1.0" />
+    </material>
+    <material name="lightgrey">
+      <color rgba="0.5 0.5 0.5 1.0" />
+    </material>
+    <material name="grey">
+      <color rgba="0.75 0.75 0.75 1.0" />
+    </material>
+    <material name="white">
+      <color rgba="0.95 0.95 0.95 1.0" />
+    </material>
+    <material name="red">
+      <color rgba="0.95 0.0 0.0 1.0" />
+    </material>
+    <material name="orange">
+      <color rgba="1.0 0.5 0.0 1.0" />
+    </material>
+    <material name="yellow">
+      <color rgba="1.0 1.0 0.0 1.0" />
+    </material>
+    <material name="green">
+      <color rgba="0.0 1.0 0.0 1.0" />
+    </material>
+    <material name="blue">
+      <color rgba="0.0 0.0 1.0 1.0" />
+    </material>
+    <material name="indigo">
+      <color rgba="0.3 0.3 0.6 1.0" />
+    </material>
+    <material name="violet">
+      <color rgba="0.6 0.0 1.0 1.0" />
+    </material>
+    <material name="black">
+      <color rgba="0.0 0.0 0.0 1.0" />
+    </material>
+    <material name="darkolive">
+      <color rgba="0.3 0.3 0.25 1.0" />
+    </material>
+  </xacro:macro>
 </robot>

Commit message: (description) add TM-s series

File: tm_description/xacro/macro.materials.xacro (robot description, xacro)
@@ -1,44 +1,44 @@
 <?xml version="1.0"?>
 <robot xmlns:xacro="http://www.ros.org/wiki/xacro">
-  <xacro:macro name="tmr_materials">
-    <material name="none">
-      <color rgba="0.0 0.0 0.0 1.0" />
-    </material>
-    <material name="lightgrey">
-      <color rgba="0.5 0.5 0.5 1.0" />
-    </material>
-    <material name="grey">
-      <color rgba="0.75 0.75 0.75 1.0" />
-    </material>
-    <material name="white">
-      <color rgba="0.95 0.95 0.95 1.0" />
-    </material>
-    <material name="red">
-      <color rgba="0.95 0.0 0.0 1.0" />
-    </material>
-    <material name="orange">
-      <color rgba="1.0 0.5 0.0 1.0" />
-    </material>
-    <material name="yellow">
-      <color rgba="1.0 1.0 0.0 1.0" />
-    </material>
-    <material name="green">
-      <color rgba="0.0 1.0 0.0 1.0" />
-    </material>
-    <material name="blue">
-      <color rgba="0.0 0.0 1.0 1.0" />
-    </material>
-    <material name="indigo">
-      <color rgba="0.3 0.3 0.6 1.0" />
-    </material>
-    <material name="violet">
-      <color rgba="0.6 0.0 1.0 1.0" />
-    </material>
-    <material name="black">
-      <color rgba="0.0 0.0 0.0 1.0" />
-    </material>
-    <material name="darkolive">
-      <color rgba="0.3 0.3 0.25 1.0" />
-    </material>
-  </xacro:macro>
+	<xacro:macro name="tmr_materials">
+		<material name="none">
+			<color rgba="0.0 0.0 0.0 1.0" />
+		</material>
+		<material name="lightgrey">
+			<color rgba="0.5 0.5 0.5 1.0" />
+		</material>
+		<material name="grey">
+			<color rgba="0.75 0.75 0.75 1.0" />
+		</material>
+		<material name="white">
+			<color rgba="0.95 0.95 0.95 1.0" />
+		</material>
+		<material name="red">
+			<color rgba="0.95 0.0 0.0 1.0" />
+		</material>
+		<material name="orange">
+			<color rgba="1.0 0.5 0.0 1.0" />
+		</material>
+		<material name="yellow">
+			<color rgba="1.0 1.0 0.0 1.0" />
+		</material>
+		<material name="green">
+			<color rgba="0.0 1.0 0.0 1.0" />
+		</material>
+		<material name="blue">
+			<color rgba="0.0 0.0 1.0 1.0" />
+		</material>
+		<material name="indigo">
+			<color rgba="0.3 0.3 0.6 1.0" />
+		</material>
+		<material name="violet">
+			<color rgba="0.6 0.0 1.0 1.0" />
+		</material>
+		<material name="black">
+			<color rgba="0.0 0.0 0.0 1.0" />
+		</material>
+		<material name="darkolive">
+			<color rgba="0.3 0.3 0.25 1.0" />
+		</material>
+	</xacro:macro>
 </robot>
