Commit message: (description) TM5S;TM7S use geometric collision models

File: tm_description/xacro/macro.tm5s-nominal.urdf.xacro (robot description, xacro)
@@ -73,6 +73,37 @@
     <collision>
       <geometry>
-        <mesh filename="package://tm_description/meshes/tm5s/collision/tm5s-base_c.stl" />
-      </geometry>
+        <cylinder radius="0.0635" length="0.072"/>
+      </geometry>
+      <origin rpy="0 0 0" xyz="0 0 0.036" />
+    </collision>
+    <collision>
+      <geometry>
+        <box size="0.02 0.05 0.065"/>
+      </geometry>
+      <origin rpy="0 0 0" xyz="-0.0615 0 0.0325" />
+    </collision>
+    <collision>
+      <geometry>
+        <box size="0.177 0.025 0.01"/>
+      </geometry>
+      <origin rpy="0 0 ${radians(45)}" xyz="0 0 0.005" />
+    </collision>
+    <collision>
+      <geometry>
+        <box size="0.177 0.025 0.01"/>
+      </geometry>
+      <origin rpy="0 0 ${radians(-45)}" xyz="0 0 0.005" />
+    </collision>
+    <collision>
+      <geometry>
+        <box size="0.143 0.1075 0.01"/>
+      </geometry>
+      <origin rpy="0 0 0" xyz="0 0 0.005" />
+    </collision>
+    <collision>
+      <geometry>
+        <box size="0.1075 0.143 0.01"/>
+      </geometry>
+      <origin rpy="0 0 0" xyz="0 0 0.005" />
     </collision>
 <!--inertial-->
@@ -101,6 +132,13 @@
     <collision>
       <geometry>
-        <mesh filename="package://tm_description/meshes/tm5s/collision/tm5s-j1_c.stl" />
-      </geometry>
+        <cylinder radius="0.0635" length="0.17475"/>
+      </geometry>
+      <origin rpy="0 0 0" xyz="0 0 0.00275" />
+    </collision>
+    <collision>
+      <geometry>
+        <cylinder radius="0.0635" length="0.07"/>
+      </geometry>
+      <origin rpy="${radians(90)} 0 0" xyz="0 -0.037 0" />
     </collision>
     <inertial>
@@ -130,6 +168,19 @@
     <collision>
       <geometry>
-        <mesh filename="package://tm_description/meshes/tm5s/collision/tm5s-a1_c.stl" />
-      </geometry>
+        <cylinder radius="0.0635" length="0.17475"/>
+      </geometry>
+      <origin rpy="0 0 0" xyz="0 0 -0.15175" />
+    </collision>
+    <collision>
+      <geometry>
+        <cylinder radius="0.0635" length="0.429"/>
+      </geometry>
+      <origin rpy="0 ${radians(90)} 0" xyz="${0.429/2} 0 -0.15" />
+    </collision>
+    <collision>
+      <geometry>
+        <cylinder radius="0.0635" length="0.17475"/>
+      </geometry>
+      <origin rpy="0 0 0" xyz="0.429 0 -0.15175" />
     </collision>
     <inertial>
@@ -159,6 +210,19 @@
     <collision>
       <geometry>
-        <mesh filename="package://tm_description/meshes/tm5s/collision/tm5s-a2_c.stl" />
-      </geometry>
+        <cylinder radius="0.0635" length="0.101"/>
+      </geometry>
+      <origin rpy="0 0 0" xyz="0 0 -0.022" />
+    </collision>
+    <collision>
+      <geometry>
+        <cylinder radius="0.044" length="0.386"/>
+      </geometry>
+      <origin rpy="0 ${radians(90)} 0" xyz="${0.386/2} 0 -0.01625" />
+    </collision>
+    <collision>
+      <geometry>
+        <cylinder radius="0.05" length="0.136"/>
+      </geometry>
+      <origin rpy="0 0 0" xyz="0.386 0 -0.022" />
     </collision>
     <inertial>
@@ -188,6 +252,13 @@
     <collision>
       <geometry>
-        <mesh filename="package://tm_description/meshes/tm5s/collision/tm5s-j5_c.stl" />
-      </geometry>
+        <cylinder radius="0.05" length="0.06"/>
+      </geometry>
+      <origin rpy="0 0 0" xyz="0 0 0.031" />
+    </collision>
+    <collision>
+      <geometry>
+        <cylinder radius="0.05" length="0.135"/>
+      </geometry>
+      <origin rpy="${radians(90)} 0 0" xyz="0 -0.0055 0" />
     </collision>
     <inertial>
@@ -217,6 +288,13 @@
     <collision>
       <geometry>
-        <mesh filename="package://tm_description/meshes/tm5s/collision/tm5s-j6_c.stl" />
-      </geometry>
+        <cylinder radius="0.05" length="0.06"/>
+      </geometry>
+      <origin rpy="0 0 0" xyz="0 0 -0.031" />
+    </collision>
+    <collision>
+      <geometry>
+        <cylinder radius="0.05" length="0.135"/>
+      </geometry>
+      <origin rpy="${radians(90)} 0 0" xyz="0 -0.0055 0" />
     </collision>
     <inertial>
@@ -246,6 +324,13 @@
     <collision>
       <geometry>
-        <mesh filename="package://tm_description/meshes/tm5s/collision/tm5s-io_c.stl" />
-      </geometry>
+        <cylinder radius="0.05" length="0.065"/>
+      </geometry>
+      <origin rpy="0 0 0" xyz="0 0 -0.032" />
+    </collision>
+    <collision>
+      <geometry>
+        <box size="0.075 0.059 0.1175"/>
+      </geometry>
+      <origin rpy="0 0 0" xyz="-0.001 0.076 -0.008" />
     </collision>
     <inertial>

File: tm_description/xacro/macro.tm7s-nominal.urdf.xacro (robot description, xacro)
@@ -73,6 +73,37 @@
     <collision>
       <geometry>
-        <mesh filename="package://tm_description/meshes/tm7s/collision/tm7s-base_c.stl" />
-      </geometry>
+        <cylinder radius="0.0635" length="0.072"/>
+      </geometry>
+      <origin rpy="0 0 0" xyz="0 0 0.036" />
+    </collision>
+    <collision>
+      <geometry>
+        <box size="0.02 0.05 0.065"/>
+      </geometry>
+      <origin rpy="0 0 0" xyz="-0.0615 0 0.0325" />
+    </collision>
+    <collision>
+      <geometry>
+        <box size="0.177 0.025 0.01"/>
+      </geometry>
+      <origin rpy="0 0 ${radians(45)}" xyz="0 0 0.005" />
+    </collision>
+    <collision>
+      <geometry>
+        <box size="0.177 0.025 0.01"/>
+      </geometry>
+      <origin rpy="0 0 ${radians(-45)}" xyz="0 0 0.005" />
+    </collision>
+    <collision>
+      <geometry>
+        <box size="0.143 0.1075 0.01"/>
+      </geometry>
+      <origin rpy="0 0 0" xyz="0 0 0.005" />
+    </collision>
+    <collision>
+      <geometry>
+        <box size="0.1075 0.143 0.01"/>
+      </geometry>
+      <origin rpy="0 0 0" xyz="0 0 0.005" />
     </collision>
 <!--inertial-->
@@ -101,6 +132,13 @@
     <collision>
       <geometry>
-        <mesh filename="package://tm_description/meshes/tm7s/collision/tm7s-j1_c.stl" />
-      </geometry>
+        <cylinder radius="0.0635" length="0.17475"/>
+      </geometry>
+      <origin rpy="0 0 0" xyz="0 0 0.00275" />
+    </collision>
+    <collision>
+      <geometry>
+        <cylinder radius="0.0635" length="0.07"/>
+      </geometry>
+      <origin rpy="${radians(90)} 0 0" xyz="0 -0.037 0" />
     </collision>
     <inertial>
@@ -130,6 +168,19 @@
     <collision>
       <geometry>
-        <mesh filename="package://tm_description/meshes/tm7s/collision/tm7s-a1_c.stl" />
-      </geometry>
+        <cylinder radius="0.0635" length="0.17475"/>
+      </geometry>
+      <origin rpy="0 0 0" xyz="0 0 -0.15175" />
+    </collision>
+    <collision>
+      <geometry>
+        <cylinder radius="0.0635" length="0.329"/>
+      </geometry>
+      <origin rpy="0 ${radians(90)} 0" xyz="${0.329/2} 0 -0.15" />
+    </collision>
+    <collision>
+      <geometry>
+        <cylinder radius="0.0635" length="0.17475"/>
+      </geometry>
+      <origin rpy="0 0 0" xyz="0.329 0 -0.15175" />
     </collision>
     <inertial>
@@ -159,6 +210,19 @@
     <collision>
       <geometry>
-        <mesh filename="package://tm_description/meshes/tm7s/collision/tm7s-a2_c.stl" />
-      </geometry>
+        <cylinder radius="0.0635" length="0.101"/>
+      </geometry>
+      <origin rpy="0 0 0" xyz="0 0 -0.022" />
+    </collision>
+    <collision>
+      <geometry>
+        <cylinder radius="0.044" length="0.298"/>
+      </geometry>
+      <origin rpy="0 ${radians(90)} 0" xyz="${0.298/2} 0 -0.01625" />
+    </collision>
+    <collision>
+      <geometry>
+        <cylinder radius="0.05" length="0.136"/>
+      </geometry>
+      <origin rpy="0 0 0" xyz="0.298 0 -0.022" />
     </collision>
     <inertial>
@@ -188,6 +252,13 @@
     <collision>
       <geometry>
-        <mesh filename="package://tm_description/meshes/tm7s/collision/tm7s-j5_c.stl" />
-      </geometry>
+        <cylinder radius="0.05" length="0.06"/>
+      </geometry>
+      <origin rpy="0 0 0" xyz="0 0 0.031" />
+    </collision>
+    <collision>
+      <geometry>
+        <cylinder radius="0.05" length="0.135"/>
+      </geometry>
+      <origin rpy="${radians(90)} 0 0" xyz="0 -0.0055 0" />
     </collision>
     <inertial>
@@ -217,6 +288,13 @@
     <collision>
       <geometry>
-        <mesh filename="package://tm_description/meshes/tm7s/collision/tm7s-j6_c.stl" />
-      </geometry>
+        <cylinder radius="0.05" length="0.06"/>
+      </geometry>
+      <origin rpy="0 0 0" xyz="0 0 -0.031" />
+    </collision>
+    <collision>
+      <geometry>
+        <cylinder radius="0.05" length="0.135"/>
+      </geometry>
+      <origin rpy="${radians(90)} 0 0" xyz="0 -0.0055 0" />
     </collision>
     <inertial>
@@ -246,6 +324,13 @@
     <collision>
       <geometry>
-        <mesh filename="package://tm_description/meshes/tm7s/collision/tm7s-io_c.stl" />
-      </geometry>
+        <cylinder radius="0.05" length="0.065"/>
+      </geometry>
+      <origin rpy="0 0 0" xyz="0 0 -0.032" />
+    </collision>
+    <collision>
+      <geometry>
+        <box size="0.075 0.059 0.1175"/>
+      </geometry>
+      <origin rpy="0 0 0" xyz="-0.001 0.076 -0.008" />
     </collision>
     <inertial>

Commit message: (description) TM5S;TM7S update geometric collision models

File: tm_description/xacro/macro.tm5s-nominal.urdf.xacro (robot description, xacro)
@@ -105,25 +105,25 @@
     <collision>
       <geometry>
-        <box size="0.177 0.025 0.01"/>
-      </geometry>
-      <origin rpy="0 0 ${radians(45)}" xyz="0 0 0.005" />
-    </collision>
-    <collision>
-      <geometry>
-        <box size="0.177 0.025 0.01"/>
-      </geometry>
-      <origin rpy="0 0 ${radians(-45)}" xyz="0 0 0.005" />
-    </collision>
-    <collision>
-      <geometry>
-        <box size="0.143 0.1075 0.01"/>
-      </geometry>
-      <origin rpy="0 0 0" xyz="0 0 0.005" />
-    </collision>
-    <collision>
-      <geometry>
-        <box size="0.1075 0.143 0.01"/>
-      </geometry>
-      <origin rpy="0 0 0" xyz="0 0 0.005" />
+        <box size="0.177 0.025 0.012"/>
+      </geometry>
+      <origin rpy="0 0 ${radians(45)}" xyz="0 0 0.006" />
+    </collision>
+    <collision>
+      <geometry>
+        <box size="0.177 0.025 0.012"/>
+      </geometry>
+      <origin rpy="0 0 ${radians(-45)}" xyz="0 0 0.006" />
+    </collision>
+    <collision>
+      <geometry>
+        <box size="0.143 0.1075 0.012"/>
+      </geometry>
+      <origin rpy="0 0 0" xyz="0 0 0.006" />
+    </collision>
+    <collision>
+      <geometry>
+        <box size="0.1075 0.143 0.012"/>
+      </geometry>
+      <origin rpy="0 0 0" xyz="0 0 0.006" />
     </collision>
 <!--inertial-->

File: tm_description/xacro/macro.tm7s-nominal.urdf.xacro (robot description, xacro)
@@ -105,25 +105,25 @@
     <collision>
       <geometry>
-        <box size="0.177 0.025 0.01"/>
-      </geometry>
-      <origin rpy="0 0 ${radians(45)}" xyz="0 0 0.005" />
-    </collision>
-    <collision>
-      <geometry>
-        <box size="0.177 0.025 0.01"/>
-      </geometry>
-      <origin rpy="0 0 ${radians(-45)}" xyz="0 0 0.005" />
-    </collision>
-    <collision>
-      <geometry>
-        <box size="0.143 0.1075 0.01"/>
-      </geometry>
-      <origin rpy="0 0 0" xyz="0 0 0.005" />
-    </collision>
-    <collision>
-      <geometry>
-        <box size="0.1075 0.143 0.01"/>
-      </geometry>
-      <origin rpy="0 0 0" xyz="0 0 0.005" />
+        <box size="0.177 0.025 0.012"/>
+      </geometry>
+      <origin rpy="0 0 ${radians(45)}" xyz="0 0 0.006" />
+    </collision>
+    <collision>
+      <geometry>
+        <box size="0.177 0.025 0.012"/>
+      </geometry>
+      <origin rpy="0 0 ${radians(-45)}" xyz="0 0 0.006" />
+    </collision>
+    <collision>
+      <geometry>
+        <box size="0.143 0.1075 0.012"/>
+      </geometry>
+      <origin rpy="0 0 0" xyz="0 0 0.006" />
+    </collision>
+    <collision>
+      <geometry>
+        <box size="0.1075 0.143 0.012"/>
+      </geometry>
+      <origin rpy="0 0 0" xyz="0 0 0.006" />
     </collision>
 <!--inertial-->
